File: PCB/rev0.2/carradio_peripheral_rev02.kicad_sch (KiCad schematic)
At the start: 209 parts, among them J1 ISO 10487 A (via pigtail), J10 Expansion, J11 SMA GNSS antenna, J12 Display buttons, J13 HDMI in (from VIM3), J14 Display FPC 40P 0.5mm, J16 Pico USB pads, J17 RTL-SDR (internal), J18 VIM3 VIN (JST-XH 2P), J19 External USB 1, J2 VIM3 40-pin via 2x20 IDC ribb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, J20 External USB 2, J3 Pico 2 pins 1-20 (1x20 F), J4 Pico 2 pins 21-40 (1x20 F), J5 VIM3 POWER key lead, J7 BH1750 light sensor, J8 ISO 10487 C1 (via pigtail), Q1 AO3400A, Q10 P-MOSFET -40V, Q11 CSD18543Q3A, Q12 CSD18543Q3A, Q2 P-MOSFET -60V, Q3 2N7002, U1 TPS560430XDBVR, U10 PCM5102APWR, U11 PCM5102APWR, U12 TPS55288RPMR, U13 CH334R, U14 CH334R, U15 LMR33630ADDA, U16 TPS2561DRCR, U17 USBLC6-2SC6, U18 USBLC6-2SC6, U2 EL817S1(C), U3 EL817S1(C), U4 EL817S1(C), U5 EL817S1(C), U6 LP5907MFX-3.3, U7 NEO-M9N-00B, U8 LP5907MFX-3.3, U9 LP5907MFX-3.3, Y1 12MHz, Y2 12MHz

Commit message: PCB rev 0.2/0.3: fix KiCad 10 footprint pad mismatches
- J13 HDMI footprint lives in Connector_Video, not Connector_HDMI
- USB-A shield pin renumbered SH to match the Molex 67643 footprint
- Hub crystals Y1/Y2 use Crystal_GND24 (pads 2/4 to GND)
- J14 FPC mounting pads (MP) tied to GND

Co-Authored-By: Claude Opus 5.5 (1M context) <noreply@anthropic.com>
Claude-Session: https://claude.ai/code/session_01C8m2AkFwQrNE2yN9Ymgjwu
Parts:
- removed J14: Display FPC 40P 0.5mm, Connector_FFC-FPC:Hirose_FH12-40S-0.5SH_1x40-1MP_P0.50mm_Horizontal, symbol Connector_Generic:Conn_01x40
- removed Y1, Y2: 12MHz, Crystal:Crystal_SMD_3225-4Pin_3.2x2.5mm, symbol Device:Crystal
- added C61: 1uF, Capacitor_SMD:C_0603_1608Metric, symbol Device:C
- added J14: Display FPC 40P 0.5mm, Connector_FFC-FPC:Hirose_FH12-40S-0.5SH_1x40-1MP_P0.50mm_Horizontal, symbol Connector_Generic_MountingPin:Conn_01x40_MountingPin
- added J19: External USB 1, Connector_USB:USB_A_Molex_67643_Horizontal, symbol Connector:USB_A
- C76: renamed from J19; value External USB 1 -> 10uF; footprint Connector_USB:USB_A_Molex_67643_Horizontal -> Capacitor_SMD:C_0805_2012Metric; symbol Connector:USB_A -> Device:C; LCSC C2798029 -> C15850; MPN Molex 67643-0910 USB-A -> 0805 10uF 25V X5R
- J13: footprint Connector_HDMI:HDMI_A_Amphenol_10029449-x01xLF_Horizontal -> Connector_Video:HDMI_A_Amphenol_10029449-x01xLF_Horizontal
- Y1: renamed from C61; value 1uF -> 12MHz; footprint Capacitor_SMD:C_0603_1608Metric -> Crystal:Crystal_SMD_3225-4Pin_3.2x2.5mm; symbol Device:C -> Device:Crystal_GND24; LCSC C77386 -> C9002; MPN 0603 1uF 50V X5R (Murata GRM188R61H105KAALD) -> YXC X322512MSB4SI 12MHz
- Y2: renamed from C76; value 10uF -> 12MHz; footprint Capacitor_SMD:C_0805_2012Metric -> Crystal:Crystal_SMD_3225-4Pin_3.2x2.5mm; symbol Device:C -> Device:Crystal_GND24; LCSC C15850 -> C9002; MPN 0805 10uF 25V X5R -> YXC X322512MSB4SI 12MHz
Connections:
- net +5V_SYS: now also C61.1, J14.4 (Pin_4), J14.5 (Pin_5), J14.6 (Pin_6); no longer Y1.1
- net BL_EN: now also J14.37 (Pin_37)
- net BL_PWM: now also J14.36 (Pin_36)
- net EXT1_DM: now also J19.2 (D-); no longer C76.2 (D-)
- net EXT1_DP: now also J19.3 (D+); no longer C76.3 (D+)
- net EXT1_VBUS: now also J19.1 (VBUS); no longer C76.1 (VBUS)
- net GND: now also C76.2, J17.SH (Shield), J20.SH (Shield), Y1.4, Y2.4, C61.2, J14.10 (Pin_10), J14.12 (Pin_12), J14.15 (Pin_15), J14.18 (Pin_18), J14.21 (Pin_21), J14.26 (Pin_26), J14.35 (Pin_35), J14.8 (Pin_8), J14.9 (Pin_9), J14.MP (MountPin), J19.4 (GND), J19.SH (Shield); no longer C76.4 (GND), C76.5 (Shield), J17.5 (Shield), J20.5 (Shield)
- net HDMI_5V: now also J14.27 (Pin_27)
- net HDMI_CEC: now also J14.23 (Pin_23)
- net HDMI_CLKN: now also J14.22 (Pin_22)
- net HDMI_CLKP: now also J14.20 (Pin_20)
- net HDMI_D0N: now also J14.19 (Pin_19)
- net HDMI_D0P: now also J14.17 (Pin_17)
- net HDMI_D1N: now also J14.16 (Pin_16)
- net HDMI_D1P: now also J14.14 (Pin_14)
- net HDMI_D2N: now also J14.13 (Pin_13)
- net HDMI_D2P: now also J14.11 (Pin_11)
- net HDMI_HPD: now also J14.28 (Pin_28)
- net HDMI_SCL: now also J14.24 (Pin_24)
- net HDMI_SDA: now also J14.25 (Pin_25)
- net HUB2_3V3: now also C76.1; no longer Y2.1
- net HUB2_XI: now also Y2.1
- net HUB2_XO: now also Y2.3
- net HUB_XI: now also Y1.1
- net HUB_XO: now also Y1.3
- net TOUCH_DN: now also J14.34 (Pin_34)
- net TOUCH_DP: now also J14.33 (Pin_33)
