File: PCB/rev0.4/main/carradio_peripheral_rev04.kicad_sch (KiCad schematic)
At the start: 203 parts, among them J1 ISO 10487 A (via pigtail), J10 Expansion, J12 Display buttons, J13 HDMI in (from VIM3), J14 Display FPC 40P 0.5mm, J18 VIM3 VIN (JST-XH 2P), J2 VIM3 40-pin via 2x20 IDC ribb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, J21 Expansion 2, J22 SWD, J23 Audio module socket, J25 USB module socket, J27 GNSS module socket, J5 VIM3 POWER key lead, J7 BH1750 light sensor, J8 ISO 10487 C1 (via pigtail), Q1 AO3400A, Q10 P-MOSFET -40V, Q11 CSD18543Q3A, Q12 CSD18543Q3A, Q2 P-MOSFET -60V, Q3 2N7002, SW1 BOOTSEL, SW2 RESET, U1 TPS560430XDBVR, U12 TPS55288RPMR, U13 CH334R, U19 AP2112K-3.3, U2 EL817S1(C), U20 RP2350B, U21 W25Q128JVS, U3 EL817S1(C), U4 EL817S1(C), U5 EL817S1(C), U6 LP5907MFX-3.3, Y1 12MHz, Y3 12MHz

Commit message: PCB rev 0.4: power hub 1 from the always-on 5V so a blank MCU flashes over USB
Hub 1 (U13) ran from +5V_SYS, which only exists after the MCU firmware
enables the TPS55288, so a blank RP2350B could only be flashed over SWD.
U13 VDD and C61 now sit on +5V_AON, and R104 (10k to HUB_3V3) keeps the
hub out of reset while the blank MCU's pads default to pull-down.
README gains a flashing section.

Co-Authored-By: Claude Opus 5.5 (1M context) <noreply@anthropic.com>
Claude-Session: https://claude.ai/code/session_01C8m2AkFwQrNE2yN9Ymgjwu
Parts:
- removed R93: 10k, Resistor_SMD:R_0603_1608Metric, symbol Device:R
- removed R97: 0Ω, Resistor_SMD:R_0402_1005Metric, symbol Device:R
- added R92: 10k, Resistor_SMD:R_0603_1608Metric, symbol Device:R
- added R99: 2.2Ω 0805, Resistor_SMD:R_0805_2012Metric, symbol Device:R
- added TH1: NTC 10k B3950, Resistor_SMD:R_0603_1608Metric, symbol Device:Thermistor_NTC
- C104: renamed from R99; value 2.2Ω 0805 -> 1nF; footprint Resistor_SMD:R_0805_2012Metric -> Capacitor_SMD:C_0603_1608Metric; symbol Device:R -> Device:C; LCSC C17521 -> C1588; MPN UNI-ROYAL 0805W8F220KT5E 0805 2.2R 125mW -> Samsung CL10B102KB8NNNC 0603 1nF 50V X7R
- R104: renamed from R79; value 1k -> 10k; LCSC C21190 -> C25804; MPN 0603 1k 1% -> 0603 10k 1%
- R79: renamed from R91; value 10k -> 1k; LCSC C25804 -> C21190; MPN 0603 10k 1% -> 0603 1k 1%
- R93: renamed from TH1; value NTC 10k B3950 -> 10k; symbol Device:Thermistor_NTC -> Device:R; LCSC C13564 -> C25804; MPN Murata NCP18XH103F03RB 10k B3380 0603 -> 0603 10k 1%
- R98: renamed from C104; value 1nF -> 0Ω; footprint Capacitor_SMD:C_0603_1608Metric -> Resistor_SMD:R_0402_1005Metric; symbol Device:C -> Device:R; LCSC C1588 -> C17168; MPN Samsung CL10B102KB8NNNC 0603 1nF 50V X7R -> UNI-ROYAL 0402WGF0000TCE 0402 0R
- renumbered R92 to R91, R98 to R97
Connections:
- net +3V3_MCU: now also R93.1
- net +5V_AON: now also C61.1, U13.12 (V5)
- net +5V_SYS: now also R91.1; no longer C61.1, R79.1, U13.12 (V5)
- net BB_DR1H: now also R97.1
- net BB_DR1H_G: now also R97.2
- net BB_DR1L: now also R98.1; no longer R97.1
- net BB_DR1L_G: now also R98.2; no longer R97.2
- net BB_SNUB: now also C104.2, R99.1; no longer C104.1, R98.2
- net BB_SW1: now also C104.1; no longer R98.1
- net GND: now also R92.2, R99.2, TH1.2; no longer C104.2, R91.2, R93.2
- net GNSS_SAFEBOOT: now also R79.2; no longer R104.2
- net HUB1_RST: now also R104.2
- net HUB_3V3: now also R104.1
- net MCU_5VSYS_ADC: now also R91.2, R92.1; no longer R79.2, R91.1
- net MCU_GNSS_SAFEBOOT: now also R79.1; no longer R104.1
- net MCU_TEMP_ADC: now also R93.2, TH1.1; no longer R93.1
Other:
- note added: "5. GNSS MODULE: u-blox NEO-M9N, active antenna on U.FL (pigtail to SMA), UART + USB to the main board. Switched 3.3V supply stays on the main board."
- note added: "Hub 1 runs from the always-on +5V_AON so a blank MCU enumerates (first flash over USB). One link to the VIM3: no USB cables. Port 1 MCU, 2 touch, 3 GNSS module USB, 4 second hub (external ports + RTL-SDR). Route D+/D- as 90 ohm pairs."
- note removed: "5. GNSS MODULE: u-blox NEO-M9N, active antenna on SMA, UART + USB to the main board. Switched 3.3V supply stays on the main board."
- note removed: "One link to the VIM3: no USB cables. Port 1 MCU, 2 touch, 3 GNSS module USB, 4 second hub (external ports + RTL-SDR). Route D+/D- as 90 ohm pairs."
- moved on the sheet: R104, R79, R91, R97
Changed lines of the file:
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@@
 )
   (text
-    "5. GNSS MODULE: u-blox NEO-M9N, active antenna on SMA, UART + USB to the main board. Switched 3.3V supply stays on the main board."
+    "5. GNSS MODULE: u-blox NEO-M9N, active antenna on U.FL (pigtail to SMA), UART + USB to the main board. Switched 3.3V supply stays on the main board."
     (at 215 158 0)
     (effects
@@
 )
   (label
-    "+5V_SYS"
+    "+5V_AON"
     (at 700 269.68 90)
     (fields_autoplaced)
@@
           (unit 1)))))
   (label
-    "+5V_SYS"
+    "+5V_AON"
     (at 720 258.19 90)
     (fields_autoplaced)
@@
           (unit 1)))))
   (text
-    "One link to the VIM3: no USB cables. Port 1 MCU, 2 touch, 3 GNSS module USB, 4 second hub (external ports + RTL-SDR). Route D+/D- as 90 ohm pairs."
+    "Hub 1 runs from the always-on +5V_AON so a blank MCU enumerates (first flash over USB). One link to the VIM3: no USB cables. Port 1 MCU, 2 touch, 3 GNSS module USB, 4 second hub (external ports + RTL-SDR). Route D+/D- as 90 ohm pairs."
     (at 610 345 0)
     (effects
@@
     (fields_autoplaced)
     (effects
+      (font
+        (size 1.27 1.27))
+      (justify right bottom))
+)
+  (symbol
+    (lib_id "Device:R")
+    (at 1108 360 0)
+    (unit 1)
+    (in_bom yes)
+    (on_board yes)
+    (dnp no)
+    (fields_autoplaced)
+    (property
+      "Reference"
+      "R104"
+      (at 1110.2 358.8 0)
+      (effects
+        (font
+          (size 1.27 1.27))
+        (justify left)))
+    (property
+      "Value"
+      "10k"
+      (at 1110.2 361.2 0)
+      (effects
+        (font
+          (size 1 1))
+        (justify left)))
+    (property
+      "Footprint"
+      "Resistor_SMD:R_0603_1608Metric"
+      (at 1108 360 0)
+      (effects
+        (font
+          (size 1.27 1.27))
+        hide))
+    (property
+      "Datasheet"
+      ""
+      (at 1108 360 0)
+      (effects
+        (font
+          (size 1.27 1.27))
+        hide))
+    (property
+      "LCSC"
+      "C25804"
+      (at 1108 360 0)
+      (effects
+        (font
+          (size 1.27 1.27))
+        hide))
+    (property
+      "MPN"
+      "0603 10k 1%"
+      (at 1108 360 0)
+      (effects
+        (font
+          (size 1.27 1.27))
+        hide))
+    (pin
+      "1"
+)
+    (pin
+      "2"
+)
+    (instances
+      (project
+        "carradio_peripheral_rev04"
+        (path
+          "/3b49dff3-5af1-5299-8484-b6e3bf9b1595"
+          (reference "R104")
+          (unit 1)))))
+  (label
+    "HUB_3V3"
+    (at 1108 356.19 90)
+    (fields_autoplaced)
+    (effects
+      (font
+        (size 1.27 1.27))
+      (justify left bottom))
+)
+  (label
+    "HUB1_RST"
+    (at 1108 363.81 270)
+    (fields_autoplaced)
+    (effects

Commit message: PCB rev 0.4: re-assign RP2350B GPIOs to face their destinations, widen the MCU ring
The autorouter kept failing at the RP2350B because many signals left the
QFN on the side away from their connector. GPIOs are re-assigned
(assign.py: Hungarian assignment on pin-to-destination distance) with
the constraints kept: ADCs on GPIO40-42, GNSS on UART1 GPIO4/5, I2C on
I2C1 GPIO30/31, and a UART pair on J10 pins 2/3 (GPIO32/33) for the
future K-line board. Expansion nets are renamed after their GPIO.

Placement keeps a 2 mm free ring around the QFN (b5.py RING) and
fanmcu.py gives every MCU pin a stub and via before autorouting.
README gains the full GPIO table.

Co-Authored-By: Claude Opus 5.5 (1M context) <noreply@anthropic.com>
Claude-Session: https://claude.ai/code/session_01C8m2AkFwQrNE2yN9Ymgjwu
Connections:
- net EXP_GP32: now also J10.2 (Pin_2); no longer J21.2 (Pin_2)
- net EXP_GP33: now also J10.3 (Pin_3); no longer J21.3 (Pin_3)
- net EXP_GP34: now also J21.2 (Pin_2); no longer J21.4 (Pin_4)
- net LUX_SCL: now also U20.39 (GPIO31); no longer U20.2 (GPIO5)
- net LUX_SDA: now also U20.38 (GPIO30); no longer U20.1 (GPIO4)
- net MCU_ACC_IN: now also U20.54 (GPIO43/ADC3); no longer U20.79 (GPIO2)
- net MCU_AMP_EN: now also U20.20 (GPIO20); no longer U20.7 (GPIO9)
- net MCU_BL_EN: now also U20.77 (GPIO0); no longer U20.8 (GPIO10)
- net MCU_BL_PWM: now also U20.78 (GPIO1); no longer U20.9 (GPIO11)
- net MCU_BTN_MUTE: now also U20.16 (GPIO16); no longer U20.28 (GPIO27)
- net MCU_BTN_SCREEN: now also U20.18 (GPIO18); no longer U20.16 (GPIO16)
- net MCU_DAC_MUTE: now also U20.8 (GPIO10); no longer U20.14 (GPIO15)
- net MCU_GNSS_EN: now also U20.7 (GPIO9); no longer U20.11 (GPIO12)
- net MCU_GNSS_PPS: now also U20.80 (GPIO3); no longer U20.19 (GPIO19)
- net MCU_GNSS_RST: now also U20.4 (GPIO7); no longer U20.18 (GPIO18)
- net MCU_GNSS_RX: now also U20.2 (GPIO5); no longer U20.78 (GPIO1)
- net MCU_GNSS_SAFEBOOT: now also U20.6 (GPIO8); no longer U20.37 (GPIO29)
- net MCU_GNSS_TX: now also U20.1 (GPIO4); no longer U20.77 (GPIO0)
- net MCU_HUB_RST: now also U20.79 (GPIO2); no longer U20.54 (GPIO43/ADC3)
- net MCU_ILLUM_IN: now also U20.46 (GPIO37); no longer U20.3 (GPIO6)
- net MCU_LED: now also U20.21 (GPIO21); no longer U20.26 (GPIO25)
- net MCU_PARK_IN: now also U20.13 (GPIO14); no longer U20.4 (GPIO7)
- net MCU_PWR_KEY: now also U20.14 (GPIO15); no longer U20.6 (GPIO8)
- net MCU_REV_IN: now also U20.44 (GPIO35); no longer U20.80 (GPIO3)
- net MCU_SBC_SENSE: now also U20.3 (GPIO6); no longer U20.12 (GPIO13)
- net MCU_SERVICE: now also U20.19 (GPIO19); no longer U20.13 (GPIO14)
- net MCU_USBP_FAULT1: now also U20.48 (GPIO39); no longer U20.23 (GPIO23)
- net MCU_USBP_FAULT2: now also U20.47 (GPIO38); no longer U20.25 (GPIO24)
- net MCU_USBP_PG: now also U20.45 (GPIO36); no longer U20.27 (GPIO26)
- net MCU_VIM3_PWR_EN: now also U20.23 (GPIO23); no longer U20.36 (GPIO28)
- removed net EXP_GP20: J10.2 (Pin_2), U20.20 (GPIO20)
- removed net EXP_GP21: J10.3 (Pin_3), U20.21 (GPIO21)
- net EXP_GP30 renamed EXP_GP28
- net EXP_GP28: now also U20.36 (GPIO28); no longer U20.38 (GPIO30)
- net EXP_GP31 renamed EXP_GP13
- net EXP_GP13: now also U20.12 (GPIO13); no longer U20.39 (GPIO31)
- net EXP_GP35 renamed EXP_GP12
- net EXP_GP12: now also U20.11 (GPIO12); no longer U20.44 (GPIO35)
- net EXP_GP36 renamed EXP_GP27
- net EXP_GP27: now also U20.28 (GPIO27); no longer U20.45 (GPIO36)
- net EXP_GP37 renamed EXP_GP26
- net EXP_GP26: now also U20.27 (GPIO26); no longer U20.46 (GPIO37)
- net EXP_GP38 renamed EXP_GP25
- net EXP_GP25: now also U20.26 (GPIO25); no longer U20.47 (GPIO38)
- net EXP_GP39 renamed EXP_GP24
- net EXP_GP24: now also U20.25 (GPIO24); no longer U20.48 (GPIO39)
- new net EXP_GP11: J21.4 (Pin_4), U20.9 (GPIO11)
- new net EXP_GP29: J21.3 (Pin_3), U20.37 (GPIO29)
Other:
- note added: "3. AMPLIFIER REMOTE (+12V from ACC, MCU GP20)"
- note added: "Display buttons (to GND): GP18 screen, GP17 vol+, GP22 vol-, GP16 mute. J12."
- note added: "GPIO44-47 are unused (ADC-capable spares)."
- note added: "Input 3V-36V (runs through cranking); output 5.0V up to 5A. MCU GP23 = EN, MCU I2C1 sets OE/voltage/current limit."
- note added: "rev 0.4: GPIO map re-assigned for routing; see the README pin table. ADC: GPIO40 battery, 41 5V rail, 42 board temperature."
- note removed: "3. AMPLIFIER REMOTE (+12V from ACC, MCU GP9)"
- note removed: "Display buttons (to GND): GP16 screen, GP17 vol+, GP22 vol-, GP27 mute. J12."
- note removed: "GPIO0-29 as rev 0.2 except: GPIO40 battery ADC (was GP26), GPIO23/24 USB port faults, GPIO25 LED, GPIO26 USB supply PG,"
- note removed: "GPIO29 GNSS safeboot, GPIO30/31 on J10, GPIO32-39 on J21, GPIO41 5V rail ADC, GPIO42 board temperature, GPIO43 hub 1 reset."
- note removed: "Input 3V-36V (runs through cranking); output 5.0V up to 5A. MCU GP28 = EN, MCU I2C0 sets OE/voltage/current limit."
Changed lines of the file:
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@@
 )
   (text
-    "3. AMPLIFIER REMOTE (+12V from ACC, MCU GP9)"
+    "3. AMPLIFIER REMOTE (+12V from ACC, MCU GP20)"
     (at 425 16 0)
     (effects
@@
 )
   (label
-    "EXP_GP20"
+    "EXP_GP32"
     (at 179.92 199.92 180)
     (fields_autoplaced)
@@
 )
   (label
-    "EXP_GP21"
+    "EXP_GP33"
     (at 179.92 202.46 180)
     (fields_autoplaced)
@@
 )
   (label
-    "EXP_GP30"
+    "EXP_GP28"
     (at 179.92 205 180)
     (fields_autoplaced)
@@
           (unit 1)))))
   (label
-    "EXP_GP31"
+    "EXP_GP13"
     (at 179.92 215.16 180)
     (fields_autoplaced)
@@
           (unit 1)))))
   (text
-    "Display buttons (to GND): GP16 screen, GP17 vol+, GP22 vol-, GP27 mute. J12."
+    "Display buttons (to GND): GP18 screen, GP17 vol+, GP22 vol-, GP16 mute. J12."
     (at 425 257 0)
     (effects
@@
           (unit 1)))))
   (text
-    "Input 3V-36V (runs through cranking); output 5.0V up to 5A. MCU GP28 = EN, MCU I2C0 sets OE/voltage/current limit."
+    "Input 3V-36V (runs through cranking); output 5.0V up to 5A. MCU GP23 = EN, MCU I2C1 sets OE/voltage/current limit."
     (at 610 205 0)
     (effects
@@
           (unit 1)))))
   (label
-    "MCU_GNSS_TX"
+    "MCU_BL_EN"
     (at 977.78 90.31 0)
     (fields_autoplaced)
@@
 )
   (label
-    "MCU_GNSS_RX"
+    "MCU_BL_PWM"
     (at 977.78 92.85 0)
     (fields_autoplaced)
@@
 )
   (label
-    "MCU_ACC_IN"
+    "MCU_HUB_RST"
     (at 977.78 95.39 0)
     (fields_autoplaced)
@@
 )
   (label
-    "MCU_REV_IN"
+    "MCU_GNSS_PPS"
     (at 977.78 97.93 0)
     (fields_autoplaced)
@@
 )
   (label
-    "LUX_SDA"
+    "MCU_GNSS_TX"
     (at 977.78 100.47 0)
     (fields_autoplaced)
@@
 )
   (label
-    "LUX_SCL"
+    "MCU_GNSS_RX"
     (at 977.78 103.01 0)
     (fields_autoplaced)
@@
 )
   (label
-    "MCU_ILLUM_IN"
+    "MCU_SBC_SENSE"
     (at 977.78 105.55 0)
     (fields_autoplaced)
@@
 )
   (label
-    "MCU_PARK_IN"
+    "MCU_GNSS_RST"
     (at 977.78 108.09 0)
     (fields_autoplaced)
@@
 )
   (label
-    "MCU_PWR_KEY"
+    "MCU_GNSS_SAFEBOOT"
     (at 977.78 110.63 0)
     (fields_autoplaced)
@@
 )
   (label
-    "MCU_AMP_EN"
+    "MCU_GNSS_EN"
     (at 977.78 113.17 0)
     (fields_autoplaced)
@@
 )
   (label
-    "MCU_BL_EN"
+    "MCU_DAC_MUTE"
     (at 977.78 115.71 0)
     (fields_autoplaced)
@@
 )
   (label
-    "MCU_BL_PWM"
+    "EXP_GP11"
     (at 977.78 118.25 0)
     (fields_autoplaced)
@@
 )
   (label
-    "MCU_GNSS_EN"
+    "EXP_GP12"
     (at 977.78 120.79 0)
     (fields_autoplaced)
@@
 )
   (label
-    "MCU_SBC_SENSE"
+    "EXP_GP13"
     (at 977.78 123.33 0)
     (fields_autoplaced)
@@
 )
   (label
-    "MCU_SERVICE"
+    "MCU_PARK_IN"
     (at 977.78 125.87 0)
     (fields_autoplaced)
@@
 )
   (label
-    "MCU_DAC_MUTE"
+    "MCU_PWR_KEY"
     (at 977.78 128.41 0)
     (fields_autoplaced)
@@
 )
   (label
-    "MCU_BTN_SCREEN"
+    "MCU_BTN_MUTE"
     (at 977.78 130.95 0)
     (fields_autoplaced)
@@
 )
   (label
-    "MCU_GNSS_RST"
+    "MCU_BTN_SCREEN"
     (at 977.78 136.03 0)
     (fields_autoplaced)
@@
 )
   (label
-    "MCU_GNSS_PPS"
+    "MCU_SERVICE"
     (at 977.78 138.57 0)
     (fields_autoplaced)
@@
 )
   (label
-    "EXP_GP20"
+    "MCU_AMP_EN"
     (at 977.78 141.11 0)
     (fields_autoplaced)
@@
 )
   (label
-    "EXP_GP21"
+    "MCU_LED"
     (at 977.78 143.65 0)
     (fields_autoplaced)
@@
 )
   (label
-    "MCU_USBP_FAULT1"
+    "MCU_VIM3_PWR_EN"
     (at 977.78 148.73 0)
     (fields_autoplaced)
@@
 )
   (label
-    "MCU_USBP_FAULT2"
+    "EXP_GP24"
     (at 977.78 151.27 0)
     (fields_autoplaced)
@@
 )
   (label
-    "MCU_LED"
+    "EXP_GP25"
     (at 977.78 153.81 0)
     (fields_autoplaced)
@@
 )
   (label
-    "MCU_USBP_PG"
+    "EXP_GP26"
     (at 977.78 156.35 0)
     (fields_autoplaced)
@@
 )
   (label
-    "MCU_BTN_MUTE"
+    "EXP_GP27"
     (at 977.78 158.89 0)
     (fields_autoplaced)
@@
 )
   (label
-    "MCU_VIM3_PWR_EN"
+    "EXP_GP28"
     (at 977.78 161.43 0)
     (fields_autoplaced)
@@
 )
   (label
-    "MCU_GNSS_SAFEBOOT"
+    "EXP_GP29"
     (at 977.78 163.97 0)
     (fields_autoplaced)
@@
 )
   (label
-    "EXP_GP30"
+    "LUX_SDA"
     (at 977.78 166.51 0)
     (fields_autoplaced)
@@
 )
   (label
-    "EXP_GP31"
+    "LUX_SCL"
     (at 977.78 169.05 0)
     (fields_autoplaced)
@@
 )
   (label
-    "EXP_GP35"
+    "MCU_REV_IN"
     (at 977.78 179.21 0)
     (fields_autoplaced)
@@
 )
   (label
-    "EXP_GP36"
+    "MCU_USBP_PG"
     (at 977.78 181.75 0)
     (fields_autoplaced)
@@
 )
   (label
-    "EXP_GP37"
+    "MCU_ILLUM_IN"
     (at 977.78 184.29 0)
     (fields_autoplaced)
@@
 )
   (label
-    "EXP_GP38"
+    "MCU_USBP_FAULT2"
     (at 977.78 186.83 0)
     (fields_autoplaced)
@@
 )
   (label
-    "EXP_GP39"
+    "MCU_USBP_FAULT1"
     (at 977.78 189.37 0)
     (fields_autoplaced)
@@
 )
   (label
-    "MCU_HUB_RST"
+    "MCU_ACC_IN"
     (at 977.78 199.53 0)
     (fields_autoplaced)
@@
           (unit 1)))))
   (label
-    "EXP_GP32"
+    "EXP_GP34"
     (at 1134.92 192.38 180)
     (fields_autoplaced)
@@
 )
   (label
-    "EXP_GP33"
+    "EXP_GP29"
     (at 1134.92 194.92 180)
     (fields_autoplaced)
@@
 )
   (label
-    "EXP_GP34"
+    "EXP_GP11"
     (at 1134.92 197.46 180)
     (fields_autoplaced)
@@
 )
   (label
-    "EXP_GP35"
+    "EXP_GP12"
     (at 1134.92 200 180)
     (fields_autoplaced)
@@
 )
   (label
-    "EXP_GP36"
+    "EXP_GP27"
     (at 1134.92 202.54 180)
     (fields_autoplaced)
@@
 )
   (label
-    "EXP_GP37"
+    "EXP_GP26"
     (at 1134.92 205.08 180)
     (fields_autoplaced)
@@
 )
   (label
-    "EXP_GP38"
+    "EXP_GP25"
     (at 1134.92 207.62 180)
     (fields_autoplaced)
@@
 )
   (label
-    "EXP_GP39"
+    "EXP_GP24"
     (at 1134.92 210.16 180)
     (fields_autoplaced)
@@
 )
   (text
-    "GPIO0-29 as rev 0.2 except: GPIO40 battery ADC (was GP26), GPIO23/24 USB port faults, GPIO25 LED, GPIO26 USB supply PG,"
+    "rev 0.4: GPIO map re-assigned for routing; see the README pin table. ADC: GPIO40 battery, 41 5V rail, 42 board temperature."
     (at 860 400 0)
     (effects
@@
 )
   (text
-    "GPIO29 GNSS safeboot, GPIO30/31 on J10, GPIO32-39 on J21, GPIO41 5V rail ADC, GPIO42 board temperature, GPIO43 hub 1 reset."
+    "GPIO44-47 are unused (ADC-capable spares)."
     (at 860 404 0)
     (effects
